Commit message: Simplify collisions and add material to bipedbot URDF

File: Control/bipedbot_ws/src/bipedbot_description/urdf/bipedbot.urdf.xacro (robot description, xacro)
@@ -5,5 +5,10 @@
 <!-- Include Gazebo Parameters -->
 <xacro:include filename="$(find bipedbot_description)/urdf/bipedbot_gazebo.xacro" />
+<!-- Greyish-black material for all visuals -->
+<material name="grey_black">
+  <color rgba="0.18 0.18 0.2 1.0"/>
+</material>
 <link name="base_footprint"/>
+<!-- ========================= base_link ========================= -->
 <link name="base_link">
   <inertial>
@@ -17,12 +22,14 @@
       <mesh filename="package://bipedbot_description/meshes/base_link.stl" scale="0.001 0.001 0.001"/>
     </geometry>
-  </visual>
-  <collision>
-    <origin xyz="0 0 0" rpy="0 0 0"/>
-    <geometry>
-      <mesh filename="package://bipedbot_description/meshes/base_link.stl" scale="0.001 0.001 0.001"/>
-    </geometry>
-  </collision>
-</link>
+    <material name="grey_black"/>
+  </visual>
+  <collision>
+    <origin xyz="0.0000 0.0107 0.1998" rpy="-1.5649 0.0000 3.1416"/>
+    <geometry>
+      <box size="0.0875 0.0907 0.1418"/>
+    </geometry>
+  </collision>
+</link>
+<!-- ========================= legs ========================= -->
 <link name="right_top_leg_1">
   <inertial>
@@ -36,9 +43,10 @@
       <mesh filename="package://bipedbot_description/meshes/right_top_leg_1.stl" scale="0.001 0.001 0.001"/>
     </geometry>
-  </visual>
-  <collision>
-    <origin xyz="-0.04 0.01 -0.199931" rpy="0 0 0"/>
-    <geometry>
-      <mesh filename="package://bipedbot_description/meshes/right_top_leg_1.stl" scale="0.001 0.001 0.001"/>
+    <material name="grey_black"/>
+  </visual>
+  <collision>
+    <origin xyz="0.0125 -0.0365 -0.0256" rpy="-2.1817 0.0000 -3.1416"/>
+    <geometry>
+      <box size="0.0250 0.0668 0.1560"/>
     </geometry>
   </collision>
@@ -55,9 +63,10 @@
       <mesh filename="package://bipedbot_description/meshes/right_bottom_leg_1.stl" scale="0.001 0.001 0.001"/>
     </geometry>
-  </visual>
-  <collision>
-    <origin xyz="-0.04 0.089867 -0.144007" rpy="0 0 0"/>
-    <geometry>
-      <mesh filename="package://bipedbot_description/meshes/right_bottom_leg_1.stl" scale="0.001 0.001 0.001"/>
+    <material name="grey_black"/>
+  </visual>
+  <collision>
+    <origin xyz="-0.0050 0.0358 -0.0512" rpy="0.6109 0.0000 0.0000"/>
+    <geometry>
+      <box size="0.0100 0.0500 0.1750"/>
     </geometry>
   </collision>
@@ -74,9 +83,10 @@
       <mesh filename="package://bipedbot_description/meshes/left_top_leg_1.stl" scale="0.001 0.001 0.001"/>
     </geometry>
-  </visual>
-  <collision>
-    <origin xyz="0.04 0.01 -0.199931" rpy="0 0 0"/>
-    <geometry>
-      <mesh filename="package://bipedbot_description/meshes/left_top_leg_1.stl" scale="0.001 0.001 0.001"/>
+    <material name="grey_black"/>
+  </visual>
+  <collision>
+    <origin xyz="-0.0125 -0.0365 -0.0256" rpy="-2.1817 0.0000 -3.1416"/>
+    <geometry>
+      <box size="0.0250 0.0668 0.1560"/>
     </geometry>
   </collision>
@@ -93,12 +103,14 @@
       <mesh filename="package://bipedbot_description/meshes/left_bottom_leg_1.stl" scale="0.001 0.001 0.001"/>
     </geometry>
-  </visual>
-  <collision>
-    <origin xyz="0.04 0.089867 -0.144007" rpy="0 0 0"/>
-    <geometry>
-      <mesh filename="package://bipedbot_description/meshes/left_bottom_leg_1.stl" scale="0.001 0.001 0.001"/>
-    </geometry>
-  </collision>
-</link>
+    <material name="grey_black"/>
+  </visual>
+  <collision>
+    <origin xyz="0.0050 0.0358 -0.0512" rpy="0.6109 0.0000 0.0000"/>
+    <geometry>
+      <box size="0.0100 0.0500 0.1750"/>
+    </geometry>
+  </collision>
+</link>
+<!-- ========================= motors ========================= -->
 <link name="right_motor_1">
   <inertial>
@@ -112,9 +124,10 @@
       <mesh filename="package://bipedbot_description/meshes/right_motor_1.stl" scale="0.001 0.001 0.001"/>
     </geometry>
-  </visual>
-  <collision>
-    <origin xyz="-0.035 0.015302 -0.037518" rpy="0 0 0"/>
-    <geometry>
-      <mesh filename="package://bipedbot_description/meshes/right_motor_1.stl" scale="0.001 0.001 0.001"/>
+    <material name="grey_black"/>
+  </visual>
+  <collision>
+    <origin xyz="0.0100 0.0000 0.0000" rpy="1.5708 0.4303 -1.5708"/>
+    <geometry>
+      <box size="0.0300 0.0300 0.0450"/>
     </geometry>
   </collision>
@@ -131,12 +144,14 @@
       <mesh filename="package://bipedbot_description/meshes/left_motor_1.stl" scale="0.001 0.001 0.001"/>
     </geometry>
-  </visual>
-  <collision>
-    <origin xyz="0.035 0.015302 -0.037518" rpy="0 0 0"/>
-    <geometry>
-      <mesh filename="package://bipedbot_description/meshes/left_motor_1.stl" scale="0.001 0.001 0.001"/>
-    </geometry>
-  </collision>
-</link>
+    <material name="grey_black"/>
+  </visual>
+  <collision>
+    <origin xyz="-0.0100 0.0000 0.0000" rpy="1.5708 -0.6891 -1.5708"/>
+    <geometry>
+      <box size="0.0300 0.0300 0.0450"/>
+    </geometry>
+  </collision>
+</link>
+<!-- ========================= wheels (no collision, tyres handle contact) ========================= -->
 <link name="left_wheel_1">
   <inertial>
@@ -150,11 +165,6 @@
       <mesh filename="package://bipedbot_description/meshes/left_wheel_1.stl" scale="0.001 0.001 0.001"/>
     </geometry>
-  </visual>
-  <collision>
-    <origin xyz="0.06 0.015302 -0.037518" rpy="0 0 0"/>
-    <geometry>
-      <mesh filename="package://bipedbot_description/meshes/left_wheel_1.stl" scale="0.001 0.001 0.001"/>
-    </geometry>
-  </collision>
+    <material name="grey_black"/>
+  </visual>
 </link>
 <link name="right_wheel_1">
@@ -169,12 +179,8 @@
       <mesh filename="package://bipedbot_description/meshes/right_wheel_1.stl" scale="0.001 0.001 0.001"/>
     </geometry>
-  </visual>
-  <collision>
-    <origin xyz="-0.06 0.015302 -0.037518" rpy="0 0 0"/>
-    <geometry>
-      <mesh filename="package://bipedbot_description/meshes/right_wheel_1.stl" scale="0.001 0.001 0.001"/>
-    </geometry>
-  </collision>
-</link>
+    <material name="grey_black"/>
+  </visual>
+</link>
+<!-- ========================= IMU (no collision) ========================= -->
 <link name="imu_link_1">
   <inertial>
@@ -188,12 +194,8 @@
       <mesh filename="package://bipedbot_description/meshes/imu_link_1.stl" scale="0.001 0.001 0.001"/>
     </geometry>
-  </visual>
-  <collision>
-    <origin xyz="-0.008 0.0055 -0.215" rpy="0 0 0"/>
-    <geometry>
-      <mesh filename="package://bipedbot_description/meshes/imu_link_1.stl" scale="0.001 0.001 0.001"/>
-    </geometry>
-  </collision>
-</link>
+    <material name="grey_black"/>
+  </visual>
+</link>
+<!-- ========================= tyres (ground contact) ========================= -->
 <link name="left_tyre_1">
   <inertial>
@@ -207,9 +209,10 @@
       <mesh filename="package://bipedbot_description/meshes/left_tyre_1.stl" scale="0.001 0.001 0.001"/>
     </geometry>
-  </visual>
-  <collision>
-    <origin xyz="0.06 0.015302 -0.037518" rpy="0 0 0"/>
-    <geometry>
-      <mesh filename="package://bipedbot_description/meshes/left_tyre_1.stl" scale="0.001 0.001 0.001"/>
+    <material name="grey_black"/>
+  </visual>
+  <collision>
+    <origin xyz="0 0 0" rpy="0 1.5708 0"/>
+    <geometry>
+      <cylinder radius="0.037" length="0.0286"/>
     </geometry>
   </collision>
@@ -226,16 +229,20 @@
       <mesh filename="package://bipedbot_description/meshes/right_tyre_1.stl" scale="0.001 0.001 0.001"/>
     </geometry>
-  </visual>
-  <collision>
-    <origin xyz="-0.06 0.015302 -0.037518" rpy="0 0 0"/>
-    <geometry>
-      <mesh filename="package://bipedbot_description/meshes/right_tyre_1.stl" scale="0.001 0.001 0.001"/>
-    </geometry>
-  </collision>
-</link>
+    <material name="grey_black"/>
+  </visual>
+  <collision>
+    <origin xyz="0 0 0" rpy="0 1.5708 0"/>
+    <geometry>
+      <cylinder radius="0.037" length="0.0286"/>
+    </geometry>
+  </collision>
+</link>
+<!-- ========================= joints ========================= -->
+<!-- z was 0.033: wheel axle is 0.0375 above base_link and tyre radius is 0.037,
+     so with z=0 the tyres sit on the ground. Verify in Gazebo. -->
 <joint name="base_joint" type="fixed">
   <parent link="base_footprint"/>
   <child link="base_link" />
-  <origin xyz="0 0 0.033" rpy="0 0 0"/>
+  <origin xyz="0 0 0" rpy="0 0 0"/>
 </joint>
 <joint name="right_top_leg_joint" type="fixed">

File: Control/bipedbot_ws/src/bipedbot_description/urdf/bipedbot_gazebo.xacro (robot description, xacro)
@@ -2,21 +2,17 @@
 <robot name="bipedbot" xmlns:xacro="http://ros.org/wiki/xacro">
     <!-- Wheels -->
-    <gazebo reference="left_wheel_1">
-        <mu1>1000000000000000.0</mu1>
-        <mu2>1000000000000000.0</mu2>
-        <kp>1000000000000.0</kp>
+    <gazebo reference="left_tyre_1">
+        <mu1>1.0</mu1>
+        <mu2>1.0</mu2>
+        <kp>100000.0</kp>
         <kd>10.0</kd>
         <minDepth>0.001</minDepth>
-        <maxVel>0.1</maxVel>
-        <fdir1>1 0 0</fdir1>
     </gazebo>
-    <gazebo reference="right_wheel_1">
-        <mu1>1000000000000000.0</mu1>
-        <mu2>1000000000000000.0</mu2>
-        <kp>1000000000000.0</kp>
+    <gazebo reference="right_tyre_1">
+        <mu1>1.0</mu1>
+        <mu2>1.0</mu2>
+        <kp>100000.0</kp>
         <kd>10.0</kd>
         <minDepth>0.001</minDepth>
-        <maxVel>0.1</maxVel>
-        <fdir1>1 0 0</fdir1>
     </gazebo>
 </robot>

Commit message: feat(description): revolute leg joints with position interfaces

File: Control/bipedbot_ws/src/bipedbot_description/urdf/bipedbot.urdf.xacro (robot description, xacro)
@@ -249,27 +249,33 @@
   <origin xyz="0 0 0" rpy="0 0 0"/>
 </joint>
-<joint name="right_top_leg_joint" type="fixed">
+<!-- Leg joints: planar hip/knee, axes parallel to the wheel axle (x). Limits cover a hip height
+     of about 0.09 .. 0.21 m (see analysis/leg_model.py); the controller restricts it further. -->
+<joint name="right_top_leg_joint" type="revolute">
   <origin xyz="0.04 -0.01 0.199931" rpy="0 0 0"/>
   <parent link="base_link"/>
   <child link="right_top_leg_1"/>
   <axis xyz="-1.0 0.0 0.0"/>
-</joint>
-<joint name="right_bottom_leg_joint" type="fixed">
+  <limit lower="-0.70" upper="0.70" effort="2.0" velocity="3.0"/>
+</joint>
+<joint name="right_bottom_leg_joint" type="revolute">
   <origin xyz="0.0 -0.079867 -0.055924" rpy="0 0 0"/>
   <parent link="right_top_leg_1"/>
   <child link="right_bottom_leg_1"/>
   <axis xyz="1.0 0.0 -0.0"/>
-</joint>
-<joint name="left_top_leg_joint" type="fixed">
+  <limit lower="-0.85" upper="0.85" effort="2.0" velocity="3.0"/>
+</joint>
+<joint name="left_top_leg_joint" type="revolute">
   <origin xyz="-0.04 -0.01 0.199931" rpy="0 0 0"/>
   <parent link="base_link"/>
   <child link="left_top_leg_1"/>
   <axis xyz="-1.0 0.0 0.0"/>
-</joint>
-<joint name="left_bottom_leg_joint" type="fixed">
+  <limit lower="-0.70" upper="0.70" effort="2.0" velocity="3.0"/>
+</joint>
+<joint name="left_bottom_leg_joint" type="revolute">
   <origin xyz="0.0 -0.079867 -0.055924" rpy="0 0 0"/>
   <parent link="left_top_leg_1"/>
   <child link="left_bottom_leg_1"/>
   <axis xyz="-1.0 0.0 -0.0"/>
+  <limit lower="-0.85" upper="0.85" effort="2.0" velocity="3.0"/>
 </joint>
 <joint name="right_motor_joint" type="fixed">

File: Control/bipedbot_ws/src/bipedbot_description/urdf/bipedbot_ros2_control.xacro (robot description, xacro)
@@ -30,4 +30,46 @@
             <state_interface name="velocity"/>
         </joint>
+        <!-- Leg joints, position-commanded. ign_ros2_control turns the position error into a
+             velocity command (gain position_proportional_gain). -->
+        <joint name="left_top_leg_joint">
+            <command_interface name="position">
+                <param name="min">-0.70</param>
+                <param name="max">0.70</param>
+            </command_interface>
+            <state_interface name="position">
+                <param name="initial_value">0.0</param>
+            </state_interface>
+            <state_interface name="velocity"/>
+        </joint>
+        <joint name="left_bottom_leg_joint">
+            <command_interface name="position">
+                <param name="min">-0.85</param>
+                <param name="max">0.85</param>
+            </command_interface>
+            <state_interface name="position">
+                <param name="initial_value">0.0</param>
+            </state_interface>
+            <state_interface name="velocity"/>
+        </joint>
+        <joint name="right_top_leg_joint">
+            <command_interface name="position">
+                <param name="min">-0.70</param>
+                <param name="max">0.70</param>
+            </command_interface>
+            <state_interface name="position">
+                <param name="initial_value">0.0</param>
+            </state_interface>
+            <state_interface name="velocity"/>
+        </joint>
+        <joint name="right_bottom_leg_joint">
+            <command_interface name="position">
+                <param name="min">-0.85</param>
+                <param name="max">0.85</param>
+            </command_interface>
+            <state_interface name="position">
+                <param name="initial_value">0.0</param>
+            </state_interface>
+            <state_interface name="velocity"/>
+        </joint>
     </ros2_control>
 </robot>
